Commit message: Update so100.urdf frame conventions for ROS 2 / REP-103
ROS 2 convention (REP-103) expects +Z as the primary rotation axis
for yaw joints and forward-axis alignment. The original OnShape export
used Y-axis joints with frame rotations baked into joint origins,
making integration with ros2_control and MoveIt non-standard.

Frame convention changes:
- Add Rz(π/2) visual rotation to base link to align meshes with
  ROS forward (+X) while keeping the joint frame Z-up
- Add Rx(π/2)+Rz(π/2) visual rotation to shoulder link so the
  mesh aligns with the reoriented shoulder frame
- Reorient shoulder inertial tensor (swap iyy/izz) to match
- Change shoulder_pan axis from Y to Z — the standard yaw axis
  in REP-103 — and remove the compensating joint rpy
- Transform shoulder_pan origin from (0,−0.0452,0.0165) to
  (0.0452,0,0.0165) to absorb the removed Rx(π/2) rotation
- Absorb Rz(π/2) into shoulder_lift rpy so downstream joints
  remain consistent without additional frame changes

Joint parameter updates:
- Effort limits: 35→2.942 N·m (actual STS3215 stall torque)
- Velocity limits: 1→5.216 rad/s (STS3215 no-load speed)

Cleanup:
- Remove ROS 1 transmission blocks

File: Simulation/SO100/so100.urdf (robot description, URDF)
Before this commit: robot so_arm100, 7 links, 6 joints
Joints:
- joint elbow_flex: limit lower=-3.14158 upper=0 effort=35 velocity=1 -> lower=-3.14158 upper=0 effort=2.942 velocity=5.21553467881118; origin xyz=0 0.11257 0.028 rpy=1.57079 0 0 -> xyz=0 0.11257 0.028 rpy=1.5707963267948966 0 0
- joint gripper: limit lower=-0.2 upper=2.0 effort=35 velocity=1 -> lower=-0.2 upper=2.0 effort=2.942 velocity=5.21553467881118; origin xyz=-0.0202 -0.0244 0 rpy=0 3.14158 0 -> xyz=-0.0202 -0.0244 0 rpy=0 3.141592653589793 0
- joint shoulder_lift: limit lower=0 upper=3.5 effort=35 velocity=1 -> lower=0 upper=3.5 effort=2.942 velocity=5.21553467881118; origin xyz=0 0.1025 0.0306 rpy=-1.8 0 0 -> xyz=0.0306 0 0.1025 rpy=-0.2292036732051035 0 1.5707963267948966
- joint shoulder_pan: axis 0 1 0 -> 0 0 1; limit lower=-2 upper=2 effort=35 velocity=1 -> lower=-2 upper=2 effort=2.942 velocity=5.21553467881118; origin xyz=0 -0.0452 0.0165 rpy=1.57079 0 0 -> xyz=0.0452 0 0.0165
- joint wrist_flex: limit lower=-2.5 upper=1.2 effort=35 velocity=1 -> lower=-2.5 upper=1.2 effort=2.942 velocity=5.21553467881118
- joint wrist_roll: limit lower=-3.14158 upper=3.14158 effort=35 velocity=1 -> lower=-3.14158 upper=3.14158 effort=2.942 velocity=5.21553467881118; origin xyz=0 -0.0601 0 rpy=0 1.57079 0 -> xyz=0 -0.0601 0 rpy=0 1.5707963267948966 0

Commit message: Add base_footprint root link to so100.urdf

File: Simulation/SO100/so100.urdf (robot description, URDF)
Before this commit: robot so_arm100, 7 links, 6 joints
Links:
- added link base_footprint
Joints:
- added joint base_footprint_joint: type fixed, parent base_footprint, child base, origin xyz=0 0 0 rpy=0 0 0

Commit message: Rename base_footprint to world in so100.urdf

File: Simulation/SO100/so100.urdf (robot description, URDF)
Before this commit: robot so_arm100, 8 links, 7 joints
Links:
- removed link base_footprint
- added link world
Joints:
- removed joint base_footprint_joint
- added joint world_joint: type fixed, parent world, child base, origin xyz=0 0 0 rpy=0 0 0

Commit message: Update so100.urdf to Z-axis joint convention for ROS 2 compatibility

File: Simulation/SO100/so100.urdf (robot description, URDF)
Before this commit: robot so_arm100, 8 links, 7 joints
Joints:
- joint elbow_flex: axis 1 0 0 -> 0 0 1; origin xyz=0 0.11257 0.028 rpy=1.5707963267948966 0 0 -> xyz=-0.028 0.11257 0 rpy=0 0 1.5707963268
- joint gripper: origin xyz=-0.0202 -0.0244 0 rpy=0 3.141592653589793 0 -> xyz=-0.0202 0 -0.0244 rpy=1.5707963268 0 3.1415926536
- joint shoulder_lift: axis 1 0 0 -> 0 0 1; origin xyz=0.0306 0 0.1025 rpy=-0.2292036732051035 0 1.5707963267948966 -> xyz=0.0306 0 0.1025 rpy=-1.5707963268 1.3415926536 0
- joint wrist_flex: axis 1 0 0 -> 0 0 1; origin xyz=0 0.0052 0.1349 rpy=-1 0 0 -> xyz=-0.1349 0.0052 0 rpy=0 0 -1
- joint wrist_roll: axis 0 1 0 -> 0 0 1; origin xyz=0 -0.0601 0 rpy=0 1.5707963267948966 0 -> xyz=0 -0.0601 0 rpy=-1.5707963268 0 0
